File: SentiBots Beta Group/Electronics Design/KiCad board/Beta Board.kicad_pcb (KiCad board)
At the start: 2 copper layers, 67.9 x 36.7 mm, 62 parts, among them P1 PWM out, P2 MCU GPIO, P3 USB OTG, P4 UART EDISON, P7 BUZZER, P8 CONN_01X02, P9 BATT, Q1 MMBT3906, U1 TXB0108PWR, U10 STM32F103CB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

Commit message: fixed minor soldermask clearance (EdiCopter)
Parts:
- added P5: GND PWM, Pin_Headers:Pin_Header_Straight_1x06, F.Cu at (113.5, 91.8)
Connections:
- P1 pad 10: GND -> 5V
- P1 pad 12: GND -> 5V
- P1 pad 2: GND -> 5V
- P1 pad 4: GND -> 5V
- P1 pad 6: GND -> 5V
- P1 pad 8: GND -> 5V
Routing:
- net 5V: track 78.1 -> 144.7 mm, vias 0 -> 1
- net GND: track 348.6 -> 351.8 mm, vias 30 -> 31
Other:
- board size 67.9 x 36.7 mm -> 69.4 x 36.8 mm
