File: SentiBots Beta Group/Electronics Design/KiCad board/Beta Board.sch (KiCad schematic (older format))
At the start: 27 parts

Commit message: added EdiCopter schematics
Parts:
- added 0.47uF1: C, symbol C
- added 1K1, 1K2: R, symbol R
- added 22uH1: INDUCTOR, symbol INDUCTOR
- added C1, C11, C16, C2, C8: 0.1uF, symbol C
- added C10: 2.2uF, symbol C
- added C12, C13: 180uF, symbol CP
- added C17: 10nF, symbol C
- added C3, C4, C6: 15uF, symbol CP
- added C5: 0.01uF, symbol C
- added C7: 1uF, symbol C
- added C9: 10uF, symbol C
- added D1: 6TQ045S, symbol D_Schottky
- added P1: PWM out, symbol CONN_02X06
- added P2: GPIO MCU, symbol CONN_01X08
- added P3: USB OTG, symbol CONN_01X05
- added P4: UART EDISON, symbol CONN_01X04
- added P5: I2C MCU, symbol CONN_01X04
- added P6: UART MCU, symbol CONN_01X04
- added R1: 100K, symbol R
- added R2: 10K, symbol R
- added R3: 536, symbol R
- added U1, U5: TXB0108PWR, symbol TXB0108PWR
- added U2: EdisonConnector, symbol EdisonConnector
- added U3: CONN_microSD, symbol CONN_microSD
- added U4: MIC2039, symbol MIC2039
- added U6: LP38691SD-3.3, symbol LP38691SD-3.3
- added U7: MIC5205-3.3YM5TR, symbol MIC5205-3.3YM5TR
- added U8: LM2678T-5.0, symbol LM2678T-5.0
- P7: renamed from P?; value CONN_01X02 -> BUZZER
- Q1: renamed from Q?; footprint SOT-23 -> (none)
- U10: renamed from U?; footprint LQFP48 -> (none)
- U9: renamed from U?; footprint QFN-24/3MM -> (none)
- gave numbers to parts that had none: 22
- renumbered R1 to R10
Connections:
- net GND: now also 0.47uF1.1, C1.2, C10.1, C11.2, C12.2, C13.2, C16.2, C17.2, C2.2, C3.2, C4.2, C6.2, C7.1, C8.1, C9.2, D1.2 (A), P1.10 (P10), P1.12 (P12), P1.2 (P2), P1.4 (P4), P1.6 (P6), P1.8 (P8), P3.5 (P5), P4.4 (P4), P5.4 (P4), P6.4 (P4), R1.2, R3.1, U1.11 (GND), U2.1 (GND), U2.11 (GND), U2.13 (GND), U2.15 (GND), U2.5 (GND), U2.9 (GND), U3.6 (GND), U4.2 (GND), U5.11 (GND), U6.2 (GND), U7.2 (GND), U8.4 (GND)
- net PWM1: now also P1.1 (P1)
- net PWM2: now also P1.3 (P3)
- net PWM3: now also P1.5 (P5)
- net PWM4: now also P1.7 (P7)
- net PWM5: now also P1.9 (P9)
- net PWN6: now also P1.11 (P11)
- net RC_CH1: now also P2.1 (P1)
- net RC_CH2: now also P2.2 (P2)
- net RC_CH3: now also P2.3 (P3)
- net RC_CH4: now also P2.4 (P4)
- net RC_CH5: now also P2.5 (P5)
- net RC_CH6: now also P2.6 (P6)
- net RC_CH7: now also P2.7 (P7)
- net RC_CH8: now also P2.8 (P8)
- net RXD: now also P6.2 (P2), U5.18 (B2)
- net SCL: now also 1K1.1, P5.1 (P1)
- net SDA: now also 1K2.1, P5.2 (P2)
- net TXD: now also P6.1 (P1), U5.20 (B1)
- net VBAT: now also 0.47uF1.2, C3.1, C4.1, C6.1, U8.2 (VIN)
- net VCC: no longer C15.1, C18.2, C20.1, C21.1, C22.1, C23.1, C24.1, D2.2 (A), D3.2 (A), D4.2 (A), P8.2 (P2), R10.1, U10.24 (VDD), U10.36 (VDD), U10.48 (VDD), U10.9 (VDDA), U9.1 (VDDIO), U9.13 (VDD), U9.8 (VDDIO)
- net VCC_IN renamed 5V
- net 5V: now also 22uH1.1, C12.1, C13.1, C7.2, C8.2, U4.1 (VIN), U6.1 (VIN_2), U6.6 (VIN), U7.1 (IN), U7.3 (EN), U8.6 (FB)
- new net: 22uH1.2, U8.1 (SW)
- new net: C5.1, U8.3 (BOOST)
- new net: C5.2, D1.1 (K)
- new net: U1.10 (OE), U1.2 (VCCA)
- new net: U1.12 (B8), U3.10 (CD)
- new net: U1.13 (B7), U3.3 (CMD/DI)
- new net: U1.14 (B6), U1.15 (B5), U3.5 (CLK)
- new net: U1.16 (B4), U3.7 (DAT0/DO)
- new net: U1.17 (B3), U3.8 (DAT1/IRQ)
- new net: U1.18 (B2), U3.1 (DAT2)
- new net: U1.20 (B1), U3.2 (DAT3/CD/CS)
- new net: R3.2, U4.5 (ILIMIT)
- new net 1.8V: C1.1, R2.2, U2.12 (1.8V), U5.10 (OE), U5.2 (VCCA)
- new net 3.3V: 1K1.2, 1K2.2, C16.1, C17.1, C2.1, C20.1, C21.1, C22.1, C23.1, C24.1, D2.2 (A), D3.2 (A), D4.2 (A), P4.3 (P3), P5.3 (P3), P6.3 (P3), P8.2 (P2), R10.1, U10.24 (VDD), U10.36 (VDD), U10.48 (VDD), U10.9 (VDDA), U2.14 (DCIN), U2.2 (VSYS), U2.4 (VSYS), U2.6 (VSYS), U3.4 (VCC), U5.19 (VCCB), U6.4 (VOUT), U6.5 (SNS)
- new net 3.3V_SEN: C11.1, C15.1, C18.2, C9.1, U7.5 (OUT), U9.1 (VDDIO), U9.13 (VDD), U9.8 (VDDIO)
- new net EDI_CTS: U2.65 (GP128_UART_1_CTS)
- new net EDI_PWM0: U2.35 (GP12_PWM0)
- new net EDI_PWM1: U2.33 (GP13_PWM1)
- new net EDI_PWM2: U2.37 (GP182_PWM2)
- new net EDI_PWM3: U2.39 (GP183_PWM3)
- new net EDI_RTX: U2.63 (GP129_UART_1_RTS)
- new net EDI_RX: U2.61 (GP130_UART_1_RX), U5.1 (A1)
- new net EDI_RX2: U2.22 (GP134_UART_2_RX), U5.5 (A4)
- new net EDI_SCL1: U2.41 (GP19_I2C_1_SCL)
- new net EDI_SCL2: U2.45 (GP27_I2C_6_SCL)
- new net EDI_SDA1: U2.43 (GP20_I2C_1_SDA)
- new net EDI_SDA2: U2.47 (GP28_I2C_6_SDA)
- new net EDI_TX: U2.46 (GP131_UART_1_TX), U5.3 (A2)
- new net EDI_TX2: U2.27 (GP135_UART_2_TX), U5.4 (A3)
- new net FAULT: R2.1, U2.19 (FAULT), U4.4 (FAULT)
- new net GPIO0: U2.24 (GP44)
- new net GPIO10: U2.59 (GP114_SPI_2_RXD)
- new net GPIO11: U2.57 (GP115_SPI_2_TXD)
- new net GPIO12: U2.55 (GP109_SPI_2_CLK)
- new net GPIO13: U2.53 (GP110_SPI_2_FS0)
- new net GPIO14: U2.51 (GP111_SPI_2_FS1)
- new net GPIO2: U2.25 (GP165)
- new net GPIO3: U2.26 (GP45)
- new net GPIO4: U2.28 (GP46)
- new net GPIO5: U2.30 (GP47)
- new net GPIO6: U2.32 (GP48)
- new net GPIO7: U2.34 (GP49)
- new net GPIO8: U2.42 (GP15)
- new net GPIO9: U2.48 (GP14)
- new net I2S_CLK: U2.52 (GP40_I2S_2_CLK)
- new net I2S_FS: U2.54 (GP41_I2S_2_FS)
- new net I2S_RXD: U2.50 (GP42_I2S_2_RXD)
- new net I2S_TXD: U2.56 (GP43_I2S_2_TXD)
- new net PSW: R1.1, U2.21 (PSW), U4.3 (ENABLE)
- new net RX2: P4.2 (P2), U5.16 (B4)
- new net SD_0_CD#: U1.9 (A8), U2.60 (GP77_SD_0_CD#)
- new net SD_0_CLK: U1.6 (A5), U2.58 (GP78_SD_0_CLK)
- new net SD_0_CMD: U1.8 (A7), U2.62 (GP79_SD_0_CMD)
- new net SD_0_DA3: U1.1 (A1), U2.68 (GP83_SD_0_DAT3)
- new net SD_0_DAT0: U1.5 (A4), U2.66 (GP80_SD_0_DAT0)
- new net SD_0_DAT1: U1.4 (A3), U2.70 (GP81_SD_0_DAT1)
- new net SD_0_DAT2: U1.3 (A2), U2.64 (GP82_SD_0_DAT2)
- new net SD_CLK_FB: U1.7 (A6), U2.44 (GP84_SD_CLK_FB)
- new net TX2: P4.1 (P1), U5.17 (B3)
- new net USB_DN: P3.2 (P2), U2.18 (USB_DN)
- new net USB_DP: P3.3 (P3), U2.16 (USB_DP)
- new net USB_ID: P3.4 (P4), U2.3 (USB_ID)
- new net V_BUS: P3.1 (P1), U2.20 (USB_VBUS), U4.6 (VOUT)
Other:
- moved on the sheet: C14, C15, C18, C19, C20, C21, C22, C23, C24, D2, D3, D4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

Commit message: finished EdiCopter rev 1
Parts:
- removed P2: GPIO MCU, symbol CONN_01X08
- removed P5: I2C MCU, symbol CONN_01X04
- removed P6: UART MCU, symbol CONN_01X04
- added P2: MCU GPIO, Pin_Headers:Pin_Header_Straight_1x16, symbol CONN_01X16
- 1K1, 1K2, R1, R10, R2, R3, R4, R5, R6, R7, R8, R9: footprint (none) -> Resistors_SMD:R_0603
- 22uH1: footprint (none) -> Inductors:NR4018
- C1, C10, C11, C12, C13, C14, C15, C16, C17, C18, C19, C2, C20, C21, C22, C23, C24, C3, C4, C5, C6, C7, C8, C9: footprint (none) -> Capacitors_SMD:C_0603
- C25: renamed from 0.47uF1; value C -> 0.47uF; footprint (none) -> Capacitors_SMD:C_0603
- D1: footprint (none) -> TO_SOT_Packages_SMD:TO-263-3Lead
- D2, D3, D4: footprint (none) -> LEDs:LED_0603
- P1: footprint (none) -> Pin_Headers:Pin_Header_Straight_2x06
- P3: footprint (none) -> Pin_Headers:Pin_Header_Straight_1x05
- P4: footprint (none) -> Pin_Headers:Pin_Header_Straight_1x04
- P7, P8, P9: footprint (none) -> Pin_Headers:Pin_Header_Straight_1x02
- Q1: footprint (none) -> TO_SOT_Packages_SMD:SOT-23
- U1, U5: footprint (none) -> TXB0108PWR:TSSOP20
- U10: footprint (none) -> Housings_QFP:LQFP-48_7x7mm_Pitch0.5mm
- U2: footprint (none) -> mogar_kicad:DF40HC(3.0)-70DS
- U3: footprint (none) -> opendous:Memory_Card_microSD_3M_290805
- U4: footprint (none) -> TO_SOT_Packages_SMD:SOT-23-6
- U6: footprint (none) -> LP38691SD-3.3:DFN300X300X80-7N
- U7: footprint (none) -> MIC5205-3.3YM5TR:SOT95P280X130-5N
- U8: footprint (none) -> manuf:TO-263-7-TEXAS
- U9: footprint (none) -> MPU-9250:QFN-24%2f3MM
- X1, X2: footprint (none) -> Crystals:Crystal_HC49-SD_SMD
Connections:
- net 3.3V: now also P2.11 (P11), P2.15 (P15)
- net GND: now also P2.12 (P12), P2.16 (P16)
- net RC_CH1: now also P2.1 (P1)
- net RC_CH2: now also P2.2 (P2)
- net RC_CH3: now also P2.3 (P3)
- net RC_CH4: now also P2.4 (P4)
- net RC_CH5: now also P2.5 (P5)
- net RC_CH6: now also P2.6 (P6)
- net RC_CH7: now also P2.7 (P7)
- net RC_CH8: now also P2.8 (P8)
- net RXD: now also P2.14 (P14)
- net SCL: now also P2.9 (P9)
- net SDA: now also P2.10 (P10)
- net TXD: now also P2.13 (P13)
- net V_BUS: now also C10.2

Commit message: fixed minor soldermask clearance (EdiCopter)
Parts:
- added P5: GND PWM, Pin_Headers:Pin_Header_Straight_1x06, symbol CONN_01X06
- added P6: logo, EdiCopter:logo, symbol CONN_01X01
Connections:
- wire segments 164 -> 166

Commit message: fixed silkscreen and added branding
Parts:
- P5: footprint Pin_Headers:Pin_Header_Straight_1x06 -> EdiCopter:Pin_Header_Straight_1x06
Changed lines of the file:
@@
 F 0 "P5" H 8750 4400 50  0000 C CNN
 F 1 "GND PWM" V 8850 4050 50  0000 C CNN
-F 2 "Pin_Headers:Pin_Header_Straight_1x06" H 8750 4050 60  0001 C CNN
+F 2 "EdiCopter:Pin_Header_Straight_1x06" H 8750 4050 60  0001 C CNN
 F 3 "" H 8750 4050 60  0000 C CNN
 	1    8750 4050
